File: can-split-keyboard.sch (KiCad schematic (older format))
At the start: 90 parts, among them SW1 SW_Push, SW10 SW_Push, SW11 SW_Push, SW12 SW_Push, SW13 SW_Push, SW14 SW_Push, SW15 SW_Push, SW16 SW_Push, SW17 SW_Push, SW18 SW_Push, SW19 SW_Push, SW2 SW_Push, SW20 SW_Push, SW21 SW_Push, SW22 SW_Push, SW23 SW_Push, SW24 SW_Push, SW25 SW_Push, SW26 SW_Push, SW27 SW_Push, SW28 SW_Push, SW29 SW_Push, SW3 SW_Push, SW30 SW_Push, SW31 SW_Push, SW32 SW_Push, SW33 SW_Push, SW34 SW_Push, SW35 SW_Push, SW36 SW_Push, SW37 SW_Push, SW38 SW_Push, SW39 SW_Push, SW4 SW_Push, SW40 SW_Push, SW41 SW_Push, SW42 SW_Push, SW5 SW_Push, SW6 SW_Push, SW7 SW_Push, SW8 SW_Push, SW9 SW_Push

Commit message: Assigned footprints to switches.
Parts:
- SW1, SW10, SW11, SW12, SW13, SW14, SW15, SW16, SW17, SW18, SW19, SW2, SW20, SW21, SW22, SW23, SW24, SW25, SW26, SW27, SW28, SW29, SW3, SW30, SW31, SW32, SW33, SW34, SW35, SW36, SW37, SW38, SW39, SW4, SW40, SW41, SW42, SW5, SW6, SW7, SW8, SW9: footprint (none) -> Peej Footprints:MX_CUTOUT
Changed lines of the file:
@@
 F 0 "SW7" H 6000 1785 50  0000 C CNN
 F 1 "SW_Push" H 6000 1694 50  0000 C CNN
-F 2 "" H 6000 1700 50  0001 C CNN
+F 2 "Peej Footprints:MX_CUTOUT" H 6000 1700 50  0001 C CNN
 F 3 "~" H 6000 1700 50  0001 C CNN
 	1    6000 1500
@@
 F 0 "SW13" H 6850 1785 50  0000 C CNN
 F 1 "SW_Push" H 6850 1694 50  0000 C CNN
-F 2 "" H 6850 1700 50  0001 C CNN
+F 2 "Peej Footprints:MX_CUTOUT" H 6850 1700 50  0001 C CNN
 F 3 "~" H 6850 1700 50  0001 C CNN
 	1    6850 1500
@@
 F 0 "SW19" H 7700 1785 50  0000 C CNN
 F 1 "SW_Push" H 7700 1694 50  0000 C CNN
-F 2 "" H 7700 1700 50  0001 C CNN
+F 2 "Peej Footprints:MX_CUTOUT" H 7700 1700 50  0001 C CNN
 F 3 "~" H 7700 1700 50  0001 C CNN
 	1    7700 1500
@@
 F 0 "SW25" H 8550 1785 50  0000 C CNN
 F 1 "SW_Push" H 8550 1694 50  0000 C CNN
-F 2 "" H 8550 1700 50  0001 C CNN
+F 2 "Peej Footprints:MX_CUTOUT" H 8550 1700 50  0001 C CNN
 F 3 "~" H 8550 1700 50  0001 C CNN
 	1    8550 1500
@@
 F 0 "SW31" H 9400 1785 50  0000 C CNN
 F 1 "SW_Push" H 9400 1694 50  0000 C CNN
-F 2 "" H 9400 1700 50  0001 C CNN
+F 2 "Peej Footprints:MX_CUTOUT" H 9400 1700 50  0001 C CNN
 F 3 "~" H 9400 1700 50  0001 C CNN
 	1    9400 1500
@@
 F 0 "SW37" H 10250 1785 50  0000 C CNN
 F 1 "SW_Push" H 10250 1694 50  0000 C CNN
-F 2 "" H 10250 1700 50  0001 C CNN
+F 2 "Peej Footprints:MX_CUTOUT" H 10250 1700 50  0001 C CNN
 F 3 "~" H 10250 1700 50  0001 C CNN
 	1    10250 1500
@@
 F 0 "SW2" H 5150 2485 50  0000 C CNN
 F 1 "SW_Push" H 5150 2394 50  0000 C CNN
-F 2 "" H 5150 2400 50  0001 C CNN
+F 2 "Peej Footprints:MX_CUTOUT" H 5150 2400 50  0001 C CNN
 F 3 "~" H 5150 2400 50  0001 C CNN
 	1    5150 2200
@@
 F 0 "SW8" H 6000 2485 50  0000 C CNN
 F 1 "SW_Push" H 6000 2394 50  0000 C CNN
-F 2 "" H 6000 2400 50  0001 C CNN
+F 2 "Peej Footprints:MX_CUTOUT" H 6000 2400 50  0001 C CNN
 F 3 "~" H 6000 2400 50  0001 C CNN
 	1    6000 2200
@@
 F 0 "SW14" H 6850 2485 50  0000 C CNN
 F 1 "SW_Push" H 6850 2394 50  0000 C CNN
-F 2 "" H 6850 2400 50  0001 C CNN
+F 2 "Peej Footprints:MX_CUTOUT" H 6850 2400 50  0001 C CNN
 F 3 "~" H 6850 2400 50  0001 C CNN
 	1    6850 2200
@@
 F 0 "SW20" H 7700 2485 50  0000 C CNN
 F 1 "SW_Push" H 7700 2394 50  0000 C CNN
-F 2 "" H 7700 2400 50  0001 C CNN
+F 2 "Peej Footprints:MX_CUTOUT" H 7700 2400 50  0001 C CNN
 F 3 "~" H 7700 2400 50  0001 C CNN
 	1    7700 2200
@@
 F 0 "SW26" H 8550 2485 50  0000 C CNN
 F 1 "SW_Push" H 8550 2394 50  0000 C CNN
-F 2 "" H 8550 2400 50  0001 C CNN
+F 2 "Peej Footprints:MX_CUTOUT" H 8550 2400 50  0001 C CNN
 F 3 "~" H 8550 2400 50  0001 C CNN
 	1    8550 2200
@@
 F 0 "SW32" H 9400 2485 50  0000 C CNN
 F 1 "SW_Push" H 9400 2394 50  0000 C CNN
-F 2 "" H 9400 2400 50  0001 C CNN
+F 2 "Peej Footprints:MX_CUTOUT" H 9400 2400 50  0001 C CNN
 F 3 "~" H 9400 2400 50  0001 C CNN
 	1    9400 2200
@@
 F 0 "SW38" H 10250 2485 50  0000 C CNN
 F 1 "SW_Push" H 10250 2394 50  0000 C CNN
-F 2 "" H 10250 2400 50  0001 C CNN
+F 2 "Peej Footprints:MX_CUTOUT" H 10250 2400 50  0001 C CNN
 F 3 "~" H 10250 2400 50  0001 C CNN
 	1    10250 2200
@@
 F 0 "SW3" H 5150 3185 50  0000 C CNN
 F 1 "SW_Push" H 5150 3094 50  0000 C CNN
-F 2 "" H 5150 3100 50  0001 C CNN
+F 2 "Peej Footprints:MX_CUTOUT" H 5150 3100 50  0001 C CNN
 F 3 "~" H 5150 3100 50  0001 C CNN
 	1    5150 2900
@@
 F 0 "SW9" H 6000 3185 50  0000 C CNN
 F 1 "SW_Push" H 6000 3094 50  0000 C CNN
-F 2 "" H 6000 3100 50  0001 C CNN
+F 2 "Peej Footprints:MX_CUTOUT" H 6000 3100 50  0001 C CNN
 F 3 "~" H 6000 3100 50  0001 C CNN
 	1    6000 2900
@@
 F 0 "SW15" H 6850 3185 50  0000 C CNN
 F 1 "SW_Push" H 6850 3094 50  0000 C CNN
-F 2 "" H 6850 3100 50  0001 C CNN
+F 2 "Peej Footprints:MX_CUTOUT" H 6850 3100 50  0001 C CNN
 F 3 "~" H 6850 3100 50  0001 C CNN
 	1    6850 2900
@@
 F 0 "SW21" H 7700 3185 50  0000 C CNN
 F 1 "SW_Push" H 7700 3094 50  0000 C CNN
-F 2 "" H 7700 3100 50  0001 C CNN
+F 2 "Peej Footprints:MX_CUTOUT" H 7700 3100 50  0001 C CNN
 F 3 "~" H 7700 3100 50  0001 C CNN
 	1    7700 2900
@@
 F 0 "SW27" H 8550 3185 50  0000 C CNN
 F 1 "SW_Push" H 8550 3094 50  0000 C CNN
-F 2 "" H 8550 3100 50  0001 C CNN
+F 2 "Peej Footprints:MX_CUTOUT" H 8550 3100 50  0001 C CNN
 F 3 "~" H 8550 3100 50  0001 C CNN
 	1    8550 2900
@@
 F 0 "SW33" H 9400 3185 50  0000 C CNN
 F 1 "SW_Push" H 9400 3094 50  0000 C CNN
-F 2 "" H 9400 3100 50  0001 C CNN
+F 2 "Peej Footprints:MX_CUTOUT" H 9400 3100 50  0001 C CNN
 F 3 "~" H 9400 3100 50  0001 C CNN
 	1    9400 2900
@@
 F 0 "SW39" H 10250 3185 50  0000 C CNN
 F 1 "SW_Push" H 10250 3094 50  0000 C CNN
-F 2 "" H 10250 3100 50  0001 C CNN
+F 2 "Peej Footprints:MX_CUTOUT" H 10250 3100 50  0001 C CNN
 F 3 "~" H 10250 3100 50  0001 C CNN
 	1    10250 2900
@@
 F 0 "SW4" H 5150 3885 50  0000 C CNN
 F 1 "SW_Push" H 5150 3794 50  0000 C CNN
-F 2 "" H 5150 3800 50  0001 C CNN
+F 2 "Peej Footprints:MX_CUTOUT" H 5150 3800 50  0001 C CNN
 F 3 "~" H 5150 3800 50  0001 C CNN
 	1    5150 3600
@@
 F 0 "SW10" H 6000 3885 50  0000 C CNN
 F 1 "SW_Push" H 6000 3794 50  0000 C CNN
-F 2 "" H 6000 3800 50  0001 C CNN
+F 2 "Peej Footprints:MX_CUTOUT" H 6000 3800 50  0001 C CNN
 F 3 "~" H 6000 3800 50  0001 C CNN
 	1    6000 3600
@@
 F 0 "SW16" H 6850 3885 50  0000 C CNN
 F 1 "SW_Push" H 6850 3794 50  0000 C CNN
-F 2 "" H 6850 3800 50  0001 C CNN
+F 2 "Peej Footprints:MX_CUTOUT" H 6850 3800 50  0001 C CNN
 F 3 "~" H 6850 3800 50  0001 C CNN
 	1    6850 3600
@@
 F 0 "SW22" H 7700 3885 50  0000 C CNN
 F 1 "SW_Push" H 7700 3794 50  0000 C CNN
-F 2 "" H 7700 3800 50  0001 C CNN
+F 2 "Peej Footprints:MX_CUTOUT" H 7700 3800 50  0001 C CNN
 F 3 "~" H 7700 3800 50  0001 C CNN
 	1    7700 3600
@@
 F 0 "SW28" H 8550 3885 50  0000 C CNN
 F 1 "SW_Push" H 8550 3794 50  0000 C CNN
-F 2 "" H 8550 3800 50  0001 C CNN
+F 2 "Peej Footprints:MX_CUTOUT" H 8550 3800 50  0001 C CNN
 F 3 "~" H 8550 3800 50  0001 C CNN
 	1    8550 3600
@@
 F 0 "SW34" H 9400 3885 50  0000 C CNN
 F 1 "SW_Push" H 9400 3794 50  0000 C CNN
-F 2 "" H 9400 3800 50  0001 C CNN
+F 2 "Peej Footprints:MX_CUTOUT" H 9400 3800 50  0001 C CNN
 F 3 "~" H 9400 3800 50  0001 C CNN
 	1    9400 3600
@@
 F 0 "SW40" H 10250 3885 50  0000 C CNN
 F 1 "SW_Push" H 10250 3794 50  0000 C CNN
-F 2 "" H 10250 3800 50  0001 C CNN
+F 2 "Peej Footprints:MX_CUTOUT" H 10250 3800 50  0001 C CNN
 F 3 "~" H 10250 3800 50  0001 C CNN
 	1    10250 3600
@@
 F 0 "SW5" H 5150 4585 50  0000 C CNN
 F 1 "SW_Push" H 5150 4494 50  0000 C CNN
-F 2 "" H 5150 4500 50  0001 C CNN
+F 2 "Peej Footprints:MX_CUTOUT" H 5150 4500 50  0001 C CNN
 F 3 "~" H 5150 4500 50  0001 C CNN
 	1    5150 4300
@@
 F 0 "SW11" H 6000 4585 50  0000 C CNN
 F 1 "SW_Push" H 6000 4494 50  0000 C CNN
-F 2 "" H 6000 4500 50  0001 C CNN
+F 2 "Peej Footprints:MX_CUTOUT" H 6000 4500 50  0001 C CNN
 F 3 "~" H 6000 4500 50  0001 C CNN
 	1    6000 4300
@@
 F 0 "SW17" H 6850 4585 50  0000 C CNN
 F 1 "SW_Push" H 6850 4494 50  0000 C CNN
-F 2 "" H 6850 4500 50  0001 C CNN
+F 2 "Peej Footprints:MX_CUTOUT" H 6850 4500 50  0001 C CNN
 F 3 "~" H 6850 4500 50  0001 C CNN
 	1    6850 4300
@@
 F 0 "SW23" H 7700 4585 50  0000 C CNN
 F 1 "SW_Push" H 7700 4494 50  0000 C CNN
-F 2 "" H 7700 4500 50  0001 C CNN
+F 2 "Peej Footprints:MX_CUTOUT" H 7700 4500 50  0001 C CNN
 F 3 "~" H 7700 4500 50  0001 C CNN
 	1    7700 4300
@@
 F 0 "SW29" H 8550 4585 50  0000 C CNN
 F 1 "SW_Push" H 8550 4494 50  0000 C CNN
-F 2 "" H 8550 4500 50  0001 C CNN
+F 2 "Peej Footprints:MX_CUTOUT" H 8550 4500 50  0001 C CNN
 F 3 "~" H 8550 4500 50  0001 C CNN
 	1    8550 4300
@@
 F 0 "SW35" H 9400 4585 50  0000 C CNN
 F 1 "SW_Push" H 9400 4494 50  0000 C CNN
-F 2 "" H 9400 4500 50  0001 C CNN
+F 2 "Peej Footprints:MX_CUTOUT" H 9400 4500 50  0001 C CNN
 F 3 "~" H 9400 4500 50  0001 C CNN
 	1    9400 4300
@@
 F 0 "SW41" H 10250 4585 50  0000 C CNN
 F 1 "SW_Push" H 10250 4494 50  0000 C CNN
-F 2 "" H 10250 4500 50  0001 C CNN
+F 2 "Peej Footprints:MX_CUTOUT" H 10250 4500 50  0001 C CNN
 F 3 "~" H 10250 4500 50  0001 C CNN
 	1    10250 4300
@@
 F 0 "SW6" H 5150 5285 50  0000 C CNN
 F 1 "SW_Push" H 5150 5194 50  0000 C CNN
-F 2 "" H 5150 5200 50  0001 C CNN
+F 2 "Peej Footprints:MX_CUTOUT" H 5150 5200 50  0001 C CNN
 F 3 "~" H 5150 5200 50  0001 C CNN
 	1    5150 5000
@@
 F 0 "SW12" H 6000 5285 50  0000 C CNN
 F 1 "SW_Push" H 6000 5194 50  0000 C CNN
-F 2 "" H 6000 5200 50  0001 C CNN
+F 2 "Peej Footprints:MX_CUTOUT" H 6000 5200 50  0001 C CNN
 F 3 "~" H 6000 5200 50  0001 C CNN
 	1    6000 5000
@@
 F 0 "SW18" H 6850 5285 50  0000 C CNN
 F 1 "SW_Push" H 6850 5194 50  0000 C CNN
-F 2 "" H 6850 5200 50  0001 C CNN
+F 2 "Peej Footprints:MX_CUTOUT" H 6850 5200 50  0001 C CNN
 F 3 "~" H 6850 5200 50  0001 C CNN
 	1    6850 5000
@@
 F 0 "SW24" H 7700 5285 50  0000 C CNN
 F 1 "SW_Push" H 7700 5194 50  0000 C CNN
-F 2 "" H 7700 5200 50  0001 C CNN
+F 2 "Peej Footprints:MX_CUTOUT" H 7700 5200 50  0001 C CNN
 F 3 "~" H 7700 5200 50  0001 C CNN
 	1    7700 5000
@@
 F 0 "SW30" H 8550 5285 50  0000 C CNN
 F 1 "SW_Push" H 8550 5194 50  0000 C CNN
-F 2 "" H 8550 5200 50  0001 C CNN
+F 2 "Peej Footprints:MX_CUTOUT" H 8550 5200 50  0001 C CNN
 F 3 "~" H 8550 5200 50  0001 C CNN
 	1    8550 5000
@@
 F 0 "SW36" H 9400 5285 50  0000 C CNN
 F 1 "SW_Push" H 9400 5194 50  0000 C CNN
-F 2 "" H 9400 5200 50  0001 C CNN
+F 2 "Peej Footprints:MX_CUTOUT" H 9400 5200 50  0001 C CNN
 F 3 "~" H 9400 5200 50  0001 C CNN
 	1    9400 5000
@@
 F 0 "SW42" H 10250 5285 50  0000 C CNN
 F 1 "SW_Push" H 10250 5194 50  0000 C CNN
-F 2 "" H 10250 5200 50  0001 C CNN
+F 2 "Peej Footprints:MX_CUTOUT" H 10250 5200 50  0001 C CNN
 F 3 "~" H 10250 5200 50  0001 C CNN
 	1    10250 5000
@@
 F 0 "SW1" H 5150 1785 50  0000 C CNN
 F 1 "SW_Push" H 5150 1694 50  0000 C CNN
-F 2 "" H 5150 1700 50  0001 C CNN
+F 2 "Peej Footprints:MX_CUTOUT" H 5150 1700 50  0001 C CNN
 F 3 "~" H 5150 1700 50  0001 C CNN
 	1    5150 1500

Commit message: Added all the footprints
Parts:
- GND1: footprint (none) -> Peej Footprints:Single_Pad
- Jack1, Jack2: footprint (none) -> Peej Footprints:PJ-320A
- Reset1: footprint (none) -> Peej Footprints:Square_Pad
Changed lines of the file:
@@
 F 0 "Jack1" H 1757 1675 50  0000 C CNN
 F 1 "AudioJack4" H 1757 1584 50  0000 C CNN
-F 2 "" H 1800 1350 50  0001 C CNN
+F 2 "Peej Footprints:PJ-320A" H 1800 1350 50  0001 C CNN
 F 3 "~" H 1800 1350 50  0001 C CNN
 	1    1800 1350
@@
 F 0 "Jack2" H 1757 2425 50  0000 C CNN
 F 1 "AudioJack4" H 1757 2334 50  0000 C CNN
-F 2 "" H 1800 2100 50  0001 C CNN
+F 2 "Peej Footprints:PJ-320A" H 1800 2100 50  0001 C CNN
 F 3 "~" H 1800 2100 50  0001 C CNN
 	1    1800 2100
@@
 F 0 "GND1" H 1780 2792 50  0000 L CNN
 F 1 "Conn_01x01" H 1780 2701 50  0000 L CNN
-F 2 "" H 1700 2750 50  0001 C CNN
+F 2 "Peej Footprints:Single_Pad" H 1700 2750 50  0001 C CNN
 F 3 "~" H 1700 2750 50  0001 C CNN
 	1    1700 2750
@@
 F 0 "Reset1" H 1780 3042 50  0000 L CNN
 F 1 "Conn_01x01" H 1780 2951 50  0000 L CNN
-F 2 "" H 1700 3000 50  0001 C CNN
+F 2 "Peej Footprints:Square_Pad" H 1700 3000 50  0001 C CNN
 F 3 "~" H 1700 3000 50  0001 C CNN
 	1    1700 3000

Commit message: Fixed footprints
Parts:
- ExtraJackData1: footprint (none) -> Peej Footprints:Single_Pad
- GND1: footprint Peej Footprints:Single_Pad -> Peej Footprints:Square_Pad
Changed lines of the file:
@@
 F 0 "ExtraJackData1" H 2980 2042 50  0000 L CNN
 F 1 "Conn_01x01" H 2980 1951 50  0000 L CNN
-F 2 "" H 2900 2000 50  0001 C CNN
+F 2 "Peej Footprints:Single_Pad" H 2900 2000 50  0001 C CNN
 F 3 "~" H 2900 2000 50  0001 C CNN
 	1    2900 2000
@@
 F 0 "GND1" H 1780 2792 50  0000 L CNN
 F 1 "Conn_01x01" H 1780 2701 50  0000 L CNN
-F 2 "Peej Footprints:Single_Pad" H 1700 2750 50  0001 C CNN
+F 2 "Peej Footprints:Square_Pad" H 1700 2750 50  0001 C CNN
 F 3 "~" H 1700 2750 50  0001 C CNN
 	1    1700 2750

Commit message: Placed all the switches on PCB.
Parts:
- SW12, SW36: footprint Peej Footprints:MX_CUTOUT -> Peej Footprints:MX
- SW42, SW6: footprint Peej Footprints:MX_CUTOUT -> Peej Footprints:MX2U_CUTOUT
Changed lines of the file:
@@
 F 0 "SW6" H 5150 5285 50  0000 C CNN
 F 1 "SW_Push" H 5150 5194 50  0000 C CNN
-F 2 "Peej Footprints:MX_CUTOUT" H 5150 5200 50  0001 C CNN
+F 2 "Peej Footprints:MX2U_CUTOUT" H 5150 5200 50  0001 C CNN
 F 3 "~" H 5150 5200 50  0001 C CNN
 	1    5150 5000
@@
 F 0 "SW12" H 6000 5285 50  0000 C CNN
 F 1 "SW_Push" H 6000 5194 50  0000 C CNN
-F 2 "Peej Footprints:MX_CUTOUT" H 6000 5200 50  0001 C CNN
+F 2 "Peej Footprints:MX" H 6000 5200 50  0001 C CNN
 F 3 "~" H 6000 5200 50  0001 C CNN
 	1    6000 5000
@@
 F 0 "SW36" H 9400 5285 50  0000 C CNN
 F 1 "SW_Push" H 9400 5194 50  0000 C CNN
-F 2 "Peej Footprints:MX_CUTOUT" H 9400 5200 50  0001 C CNN
+F 2 "Peej Footprints:MX" H 9400 5200 50  0001 C CNN
 F 3 "~" H 9400 5200 50  0001 C CNN
 	1    9400 5000
@@
 F 0 "SW42" H 10250 5285 50  0000 C CNN
 F 1 "SW_Push" H 10250 5194 50  0000 C CNN
-F 2 "Peej Footprints:MX_CUTOUT" H 10250 5200 50  0001 C CNN
+F 2 "Peej Footprints:MX2U_CUTOUT" H 10250 5200 50  0001 C CNN
 F 3 "~" H 10250 5200 50  0001 C CNN
 	1    10250 5000

Commit message: Fixed right buttom corner double key.
Parts:
- SW36: footprint Peej Footprints:MX -> Peej Footprints:MX2U_CUTOUT
- SW42: footprint Peej Footprints:MX2U_CUTOUT -> Peej Footprints:MX
Changed lines of the file:
@@
 F 0 "SW36" H 9400 5285 50  0000 C CNN
 F 1 "SW_Push" H 9400 5194 50  0000 C CNN
-F 2 "Peej Footprints:MX" H 9400 5200 50  0001 C CNN
+F 2 "Peej Footprints:MX2U_CUTOUT" H 9400 5200 50  0001 C CNN
 F 3 "~" H 9400 5200 50  0001 C CNN
 	1    9400 5000
@@
 F 0 "SW42" H 10250 5285 50  0000 C CNN
 F 1 "SW_Push" H 10250 5194 50  0000 C CNN
-F 2 "Peej Footprints:MX2U_CUTOUT" H 10250 5200 50  0001 C CNN
+F 2 "Peej Footprints:MX" H 10250 5200 50  0001 C CNN
 F 3 "~" H 10250 5200 50  0001 C CNN
 	1    10250 5000
